Commit message: added orientation limitation in rrt_ompl.py

File: urdfs/obstacle/obstacle.urdf (robot description, URDF)
Before this commit: robot obstacle, 2 links, 1 joints
Links:
- link obstacle_box: geometry collision box size=0.1 0.1 0.05; visual box size=0.1 0.1 0.05
Joints:
- joint world_to_obstacle: origin xyz=1.25 0 1 rpy=0 0 0 -> xyz=1.0 -0.3 1 rpy=0 0 0
