Commit message: new bounds and paths

File: urdfs/obstacle/saeule.urdf (robot description, URDF)
Before this commit: robot obstacle, 2 links, 1 joints
Links:
- link obstacle_box: geometry collision box size=0.05 0.05 0.4; visual box size=0.05 0.05 0.4
Joints:
- joint world_to_obstacle: origin xyz=1.3 -0.1 1.0 rpy=0 0 0 -> xyz=1.15 -0.1 1 rpy=0 0 0
