Commit message: Update URDF files and add obstacle definitions; modify joint origins and add path data for end effectors
- Adjusted joint origins in se3_object.urdf for obj_p_01 and obj_p_02 to improve alignment.
- Added new CSV files for left and right end effector paths, providing detailed trajectory data.
- Created planned_object_path.csv to define a planned trajectory for an object.
- Introduced a new obstacle.urdf file defining a fixed obstacle in the simulation environment.

File: urdfs/object/se3_object.urdf (robot description, URDF)
Before this commit: robot obj_se3, 5 links, 4 joints
Joints:
- joint virt_stick_01: origin xyz=0 -0.14 0 rpy=1.57079 3.14 1.57079 -> xyz=0 -0.18 0 rpy=0 1.57079 0
- joint virt_stick_02: origin xyz=0 0.24 0 rpy=1.57079 3.14 0.0 -> xyz=0 0.24 0 rpy=1.57079 1.57079 0.0

Commit message: fixed object orientation when rotating

File: urdfs/object/se3_object.urdf (robot description, URDF)
Before this commit: robot obj_se3, 5 links, 4 joints
Joints:
- joint virt_stick_01: origin xyz=0 -0.18 0 rpy=0 1.57079 0 -> xyz=0 -0.14 0 rpy=0 1.57079 0

File: urdfs/obstacle/obstacle.urdf (robot description, URDF)
Before this commit: robot obstacle, 2 links, 1 joints
Links:
- link obstacle_box: geometry collision box size=0.5 0.5 0.05; visual box size=0.5 0.5 0.05
Joints:
- joint world_to_obstacle: origin xyz=0.8 0 0.15 rpy=0 0 0 -> xyz=1.25 0 1 rpy=0 0 0

Commit message: Add new paths and configurations for iiwa7 robot
- Created new CSV files for left and right y-links, including y_links.csv and y_rechts.csv with detailed motion data.
- Added YAML configuration files for various paths (column2, column3, diag, regal2, rot, y) for both left and right iiwa7 robots.
- Introduced a new Python script (check_cuda.py) for diagnosing CUDA setup and environment.
- Added a URDF file (saeule2.urdf) for an obstacle model to be used in simulations.

File: urdfs/object/se3_object.urdf (robot description, URDF)
Before this commit: robot obj_se3, 5 links, 4 joints
Joints:
- joint virt_stick_01: origin xyz=0 -0.14 0 rpy=0 1.57079 0 -> xyz=0 -0.18 0 rpy=0 1.57079 1.57079

File: urdfs/obstacle/saeule.urdf (robot description, URDF)
Before this commit: robot saeule, 2 links, 1 joints
Links:
- link obstacle_box: geometry collision box size=0.05 0.05 0.3; visual box size=0.05 0.05 0.3
Joints:
- joint world_to_obstacle: origin xyz=1.15 -0.1 1 rpy=0 0 0 -> xyz=0.9 0 1 rpy=0 0 0

File: urdfs/obstacle/saeule2.urdf (robot description, URDF)
Before this commit: robot obstacle, 2 links, 1 joints
Links:
- link obstacle_box: geometry collision box size=0.05 0.05 0.4; visual box size=0.05 0.05 0.4
Joints:
- joint world_to_obstacle: origin xyz=2.2 0 1.0 rpy=0 0 0 -> xyz=1 0.1 1 rpy=0 0 0

Commit message: Add dual-arm pose debugging and RRT planning scripts with obstacle handling
- Implemented `debug_dual_arm_pose_fixed.py` for visualizing dual-arm poses using Klampt and IK.
- Created `rrt_ompl3.py` for planning paths with OMPL, including collision checking against obstacles.
- Added URDF files for obstacles (passage, passage2, regal2) to test collision avoidance in planning.
- Enhanced IK solver functions to support batch processing and improved collision checking mechanisms.
- Updated utility functions for parsing URDF files and transforming poses between different representations.

File: urdfs/object/se3_object.urdf (robot description, URDF)
Before this commit: robot obj_se3, 5 links, 4 joints
Joints:
- joint virt_stick_01: origin xyz=0 -0.18 0 rpy=0 1.57079 1.57079 -> xyz=0 -0.2 0 rpy=0 1.57079 1.57079

File: urdfs/obstacle/passage.urdf (robot description, URDF)
Before this commit: robot saeule, 2 links, 1 joints
Links:
- link obstacle_box: geometry collision box size=0.05 0.05 0.4; visual box size=0.05 0.05 0.4
Joints:
- joint world_to_obstacle: origin xyz=0.9 0 1 rpy=0 0 0 -> xyz=0.9 0.0 0.75 rpy=0 0 0

File: urdfs/obstacle/passage2.urdf (robot description, URDF)
Before this commit: robot obstacle, 2 links, 1 joints
Links:
- link obstacle_box: geometry collision box size=0.05 0.05 0.4; visual box size=0.05 0.05 0.4
Joints:
- joint world_to_obstacle: origin xyz=5.2 0 1.0 rpy=0 0 0 -> xyz=0.9 0.0 1.4 rpy=0 0 0

File: urdfs/obstacle/regal2.urdf (robot description, URDF)
Before this commit: robot obstacle, 2 links, 1 joints
Joints:
- joint world_to_obstacle: origin xyz=5.2 0 1.0 rpy=0 0 0 -> xyz=1.2 0 1.0 rpy=0 0 0
